File: cart_proj/cart_proj.kicad_sch (KiCad schematic)
At the start: 11 parts, among them CON1 GENESIS-EDGE, J1 PAD3, J2 PAD4, U1 PAL16R4, U2 74LS244, U3 74LS244, U4 GAME ROM

Commit message: Update schematics
Parts:
- removed U4: GAME ROM, symbol Custom_EPROM:27C800
- added U4: GAME ROM, symbol Custom_EPROM:27C160
Connections:
- net A20: now also U4.42 (A19)
- net A9: now also U4.41 (A8)
- net D0: now also U4.14 (Q0)
- net D1: now also U4.16 (Q1)
- net VCC: now also U4.32 (~{BYTE})
- net ~{CART_OE}: now also U4.13 (~{G})
- net ~{ROM_E}: now also U4.11 (~{E})
- net A1: now reaches CON1.A17 (A1)
- net A1: now also U4.10 (A0)
- net A8: now reaches CON1.A3 (A8)

Commit message: Update schematics
Connections:
- net D4: now also U4.23 (Q4)
- net GND: now also CON1.A1 (GND), CON1.A18 (GND), CON1.A32 (GND), U4.12 (GND), U4.31 (GND)
- net VCC: now also CON1.A2 (+5V), CON1.A31 (+5V), U4.22 (VCC)
